File: kicad/uv-led.kicad_pcb (KiCad board)
At the start: 2 copper layers, 100 x 8 mm, 10 parts, among them J1 JST_PH_B2B-PH-K_1x02_P2.00mm_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

Commit message: updated revision number on PCB silkscreen
Other:
- board text added: "UV-LED 1.1.0 Design: T. Guentzel Date: 2026-09"
- board text removed: "UV-LED 1.0 Design: T. Guentzel Date: 2026-09"
Changed lines of the file:
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@@
 		(layer "Edge.Cuts")
 	)
-	(gr_text "UV-LED 1.0\nDesign: T. Guentzel\nDate: 2026-09"
+	(gr_text "UV-LED 1.1.0\nDesign: T. Guentzel\nDate: 2026-09"
 		(at 122.6 101.8 0)
 		(layer "F.SilkS")

Commit message: added version label on silkscreen
Other:
- board text added: "UV-LED Design: T. Guentzel Date: 2026-09 Version: 1.1.0"
- board text removed: "UV-LED 1.1.0 Design: T. Guentzel Date: 2026-09"
Changed lines of the file:
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@@
 		(layer "Edge.Cuts")
 	)
-	(gr_text "UV-LED 1.1.0\nDesign: T. Guentzel\nDate: 2026-09"
-		(at 122.6 101.8 0)
+	(gr_text "UV-LED\nDesign: T. Guentzel\nDate: 2026-09\nVersion: 1.1.0"
+		(at 123.25 102.42 0)
 		(layer "F.SilkS")
 		(effects

Commit message: changed ordering of version label on silkscreen
Other:
- board text added: "UV-LED Design: T. Guentzel Version: 1.1.0 Date: 2026-09"
- board text removed: "UV-LED Design: T. Guentzel Date: 2026-09 Version: 1.1.0"
Changed lines of the file:
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@@
 		(layer "Edge.Cuts")
 	)
-	(gr_text "UV-LED\nDesign: T. Guentzel\nDate: 2026-09\nVersion: 1.1.0"
+	(gr_text "UV-LED\nDesign: T. Guentzel\nVersion: 1.1.0\nDate: 2026-09"
 		(at 123.25 102.42 0)
 		(layer "F.SilkS")

Commit message: reverted changed ordering in PCB label
Other:
- board text added: "UV-LED Design: T. Guentzel Date: 2026-09 Version: 1.1.0"
- board text removed: "UV-LED Design: T. Guentzel Version: 1.1.0 Date: 2026-09"
Changed lines of the file:
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@@
 		(layer "Edge.Cuts")
 	)
-	(gr_text "UV-LED\nDesign: T. Guentzel\nVersion: 1.1.0\nDate: 2026-09"
+	(gr_text "UV-LED\nDesign: T. Guentzel\nDate: 2026-09\nVersion: 1.1.0"
 		(at 123.25 102.42 0)
 		(layer "F.SilkS")

Commit message: added stackup and boardhouse instructions
Other:
- board text added: "Manufacturing Instruction: - Material Aluminum - Finished thickness: 1.57 mm ± 0.13 mm - PCBs must be RoHS compliant - Do not edit artwork, e.g. to add logos or order numbers - Clean to meet IPC J-STD-001E, Class 2 after assembly"

Commit message: added libraries and linked footprints
Parts:
- LOGO1: renamed from REF**; value APQ-Logo_small -> Logo_APQ; footprint footprints_project_specific:APQ-Logo_small -> Custom_footprints_project:APQ-Logo_small
Changed lines of the file:
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@@
 		(capping no)
 		(filling no)
-		(zone_defaults)
 		(pcbplotparams
 			(layerselection 0x00000000_00000000_55555555_5755f5ff)
@@
 		)
 	)
-	(footprint "footprints_project_specific:APQ-Logo_small"
+	(footprint "Custom_footprints_project:APQ-Logo_small"
 		(layer "F.Cu")
 		(at 113.5 99)
-		(property "Reference" "REF**"
-			(at 0 0 0)
-			(layer "F.SilkS")
-			(hide yes)
-			(effects
-				(font
-					(size 1 1)
-					(thickness 0.15)
-				)
-			)
-		)
-		(property "Value" "APQ-Logo_small"
-			(at 4.5 4 0)
+		(property "Reference" "LOGO1"
+			(at 0 0 0)
+			(layer "F.SilkS")
+			(hide yes)
+			(effects
+				(font
+					(size 1 1)
+					(thickness 0.15)
+				)
+			)
+		)
+		(property "Value" "Logo_APQ"
+			(at 0 4.08 0)
 			(layer "F.Fab")
 			(effects
@@
 			)
 		)
-		(attr exclude_from_pos_files exclude_from_bom)
+		(property "MFN" ""
+			(at 0 0 0)
+			(unlocked yes)
+			(layer "F.Fab")
+			(hide yes)
+			(effects
+				(font
+					(size 1 1)
+					(thickness 0.15)
+				)
+			)
+		)
+		(property "PN" ""
+			(at 0 0 0)
+			(unlocked yes)
+			(layer "F.Fab")
+			(hide yes)
+			(effects
+				(font
+					(size 1 1)
+					(thickness 0.15)
+				)
+			)
+		)
+		(property "RoHS" ""
+			(at 0 0 0)
+			(unlocked yes)
+			(layer "F.Fab")
+			(hide yes)
+			(effects
+				(font
+					(size 1 1)
+					(thickness 0.15)
+				)
+			)
+		)
+		(sheetname "/")
+		(sheetfile "uv-led.kicad_sch")
+		(units
+			(unit
+				(name "A")
+				(pins)
+			)
+		)
+		(attr exclude_from_bom)
 		(duplicate_pad_numbers_are_jumpers no)
 		(fp_circle
@@
 					(thickness 0.15)
 				)
-			)
-		)
+				(justify mirror)
+			)
+		)

Commit message: updated APQ logo footprint courtyard
Parts:
- moved LOGO1 0.50 mm to (114.0, 99.0)
Changed lines of the file:
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@@
 	(footprint "Custom_footprints_project:APQ-Logo_small"
 		(layer "F.Cu")
-		(at 113.5 99)
+		(at 114 99)
 		(property "Reference" "LOGO1"
 			(at 0 0 0)
@@
 		(sheetname "/")
 		(sheetfile "uv-led.kicad_sch")
-		(units
-			(unit
-				(name "A")
-				(pins)
-			)
-		)
 		(attr exclude_from_bom)
 		(duplicate_pad_numbers_are_jumpers no)
 		(fp_circle
 			(center 0 0)
-			(end 0.125 0)
+			(end 0.2 0)
 			(stroke
-				(width 0.25)
+				(width 0.4)
 				(type solid)
 			)
@@
 		(fp_circle
 			(center 0 1)
-			(end 0.125 1)
+			(end 0.2 1)
 			(stroke
-				(width 0.25)
+				(width 0.4)
 				(type solid)
 			)
@@
 		(fp_circle
 			(center 0 2)
-			(end 0.125 2)
+			(end 0.2 2)
 			(stroke
-				(width 0.25)
+				(width 0.4)
 				(type solid)
 			)
@@
 		(fp_circle
 			(center 1 0)
-			(end 1.125 0)
+			(end 1.2 0)
 			(stroke
-				(width 0.25)
+				(width 0.4)
 				(type solid)
 			)
@@
 		(fp_circle
 			(center 1 1)
-			(end 1.125 1)
+			(end 1.2 1)
 			(stroke
-				(width 0.25)
+				(width 0.4)
 				(type solid)
 			)
@@
 		(fp_circle
 			(center 1 2)
-			(end 1.125 2)
+			(end 1.2 2)
 			(stroke
-				(width 0.25)
+				(width 0.4)
 				(type solid)
 			)
@@
 		(fp_circle
 			(center 2 0)
-			(end 2.125 0)
+			(end 2.2 0)
 			(stroke
-				(width 0.25)
+				(width 0.4)
 				(type solid)
 			)
@@
 		(fp_circle
 			(center 2 1)
-			(end 2.125 1)
+			(end 2.2 1)
 			(stroke
-				(width 0.25)
+				(width 0.4)
 				(type solid)
 			)
@@
 		(fp_circle
 			(center 2 2)
-			(end 2.125 2)
+			(end 2.2 2)
 			(stroke
-				(width 0.25)
+				(width 0.4)
 				(type solid)
 			)
@@
 			(layer "F.SilkS")
 		)
+		(fp_rect
+			(start -0.65 -0.6)
+			(end 9.03 2.65)
+			(stroke
+				(width 0.05)
+				(type solid)
+			)
+			(fill no)
+			(layer "F.CrtYd")
+		)
 		(fp_text user "APQ"
