File: kicad/uv-led.kicad_sch (KiCad schematic)
At the start: 13 parts, among them J1 JST_PH_B2B-PH-K_1x02_P2.00mm_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

Commit message: Feature/ci pipeline (#14)
* initial addition of bom and kibot config

* replaced bom and kibot config from one inch photodetector

* added github workflows from one inch photodetector

* removed back PCB layers

* changed project files in ci.yml

* moved .github to root

* updated file paths in ci.yml

* changed screw type to M6 and increased revision to 1.1.0

* added screw model for M6

* updated revision number to 1.1.0

* updated revision number on PCB silkscreen

* added version label on silkscreen

* changed ordering of version label on silkscreen

* added badge to readme

* Fix CI version check

Fix Regex to also match a "Version:" tag at the end of string. This fixes a bug when extracting the version tag printed on the PCB.

* Bump CI to latest

* reverted changed ordering in PCB label

* updated symbol fields and added RoHs and temperature to J1 connector

* added stackup and boardhouse instructions

* added libraries and linked footprints

* Added courtyard for APQ logo

* updated APQ logo footprint courtyard

* updated physical stackup and removed back paste

---------

Co-authored-by: Patrick Baus <patrick.baus@physik.tu-darmstadt.de>
Parts:
- D1: MFN (none) -> Luminus Devices; MN SST-08-UV-A40H-F365-00 -> (none); Mfr Luminus Devices -> (none); PN (none) -> SST-08-UV-A40H-F365-00; Temperature Top = 0 °C to 125 °C -> Top = 0 °C to 100 °C
- D2, D3, D4, D5: MFN (none) -> Luminus Devices; MN SST-08-UV-A40H-F365-00 -> (none); Mfr Luminus Devices -> (none); PN (none) -> SST-08-UV-A40H-F365-00
- J1: MFN (none) -> JST Commercial; MN PH_B2B-PH-K_1x02_P2.00mm_Vertical -> (none); Mfr JST Commercial -> (none); PN (none) -> PH_B2B-PH-K_1x02_P2.00mm_Vertical; RoHS (none) -> By exemption; Temperature (none) -> Top = -25 °C to 85 °C
- LOGO3: footprint Symbol:OSHW-Logo_7.5x8mm_SilkScreen -> (none)
Changed lines of the file:
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@@
 			)
 		)
-		(property "Description" "Luminus Devices SST-08H-UV"
+		(property "Description" "UV LED 365nm"
 			(at 114.3 101.6 0)
-			(hide yes)
-			(show_name no)
-			(do_not_autoplace no)
-			(effects
-				(font
-					(size 1.27 1.27)
-				)
-			)
-		)
-		(property "MN" "SST-08-UV-A40H-F365-00 "
-			(at 114.3 101.6 90)
-			(hide yes)
-			(show_name no)
-			(do_not_autoplace no)
-			(effects
-				(font
-					(size 1.27 1.27)
-				)
-			)
-		)
-		(property "Mfr" "Luminus Devices"
-			(at 114.3 101.6 90)
 			(hide yes)
 			(show_name no)
@@
 		)
 		(property "RoHS" "Yes"
+			(at 114.3 101.6 90)
+			(hide yes)
+			(show_name no)
+			(do_not_autoplace no)
+			(effects
+				(font
+					(size 1.27 1.27)
+				)
+			)
+		)
+		(property "MFN" "Luminus Devices"
+			(at 114.3 101.6 90)
+			(hide yes)
+			(show_name no)
+			(do_not_autoplace no)
+			(effects
+				(font
+					(size 1.27 1.27)
+				)
+			)
+		)
+		(property "PN" "SST-08-UV-A40H-F365-00"
 			(at 114.3 101.6 90)
 			(hide yes)
@@
 			)
 		)
-		(property "Description" "Luminus Devices SST-08H-UV"
+		(property "Description" "UV LED 365nm"
 			(at 114.3 92.71 0)
-			(hide yes)
-			(show_name no)
-			(do_not_autoplace no)
-			(effects
-				(font
-					(size 1.27 1.27)
-				)
-			)
-		)
-		(property "MN" "SST-08-UV-A40H-F365-00 "
-			(at 114.3 92.71 90)
-			(hide yes)
-			(show_name no)
-			(do_not_autoplace no)
-			(effects
-				(font
-					(size 1.27 1.27)
-				)
-			)
-		)
-		(property "Mfr" "Luminus Devices"
-			(at 114.3 92.71 90)
 			(hide yes)
 			(show_name no)
@@
 		)
 		(property "RoHS" "Yes"
+			(at 114.3 92.71 90)
+			(hide yes)
+			(show_name no)
+			(do_not_autoplace no)
+			(effects
+				(font
+					(size 1.27 1.27)
+				)
+			)
+		)
+		(property "MFN" "Luminus Devices"
+			(at 114.3 92.71 90)
+			(hide yes)
+			(show_name no)
+			(do_not_autoplace no)
+			(effects
+				(font
+					(size 1.27 1.27)
+				)
+			)
+		)
+		(property "PN" "SST-08-UV-A40H-F365-00"
 			(at 114.3 92.71 90)
 			(hide yes)
@@
 		(exclude_from_sim no)
 		(in_bom no)
-		(on_board yes)
+		(on_board no)
 		(in_pos_files yes)
 		(dnp no)
@@
 			)
 		)
-		(property "Footprint" "Symbol:OSHW-Logo_7.5x8mm_SilkScreen"
+		(property "Footprint" ""
 			(at 278.13 173.99 0)
 			(hide yes)
@@
 			)
 		)
-		(property "Description" "Luminus Devices SST-08H-UV"
+		(property "Description" "UV LED 365nm"
 			(at 114.3 110.49 0)
-			(hide yes)
-			(show_name no)
-			(do_not_autoplace no)
-			(effects
-				(font
-					(size 1.27 1.27)
-				)
-			)
-		)
-		(property "MN" "SST-08-UV-A40H-F365-00 "
-			(at 114.3 110.49 90)
-			(hide yes)
-			(show_name no)
-			(do_not_autoplace no)
-			(effects
-				(font
-					(size 1.27 1.27)
-				)
-			)
-		)
-		(property "Mfr" "Luminus Devices"
-			(at 114.3 110.49 90)
 			(hide yes)
 			(show_name no)
@@
 		)
 		(property "RoHS" "Yes"
+			(at 114.3 110.49 90)
+			(hide yes)
+			(show_name no)
+			(do_not_autoplace no)
+			(effects
+				(font
+					(size 1.27 1.27)
+				)
+			)
+		)
+		(property "MFN" "Luminus Devices"
+			(at 114.3 110.49 90)
+			(hide yes)
+			(show_name no)
+			(do_not_autoplace no)
+			(effects
+				(font
+					(size 1.27 1.27)
+				)
+			)
+		)
+		(property "PN" "SST-08-UV-A40H-F365-00"
 			(at 114.3 110.49 90)
 			(hide yes)
@@
 			)
 		)
-		(property "MN" "PH_B2B-PH-K_1x02_P2.00mm_Vertical"
+		(property "MFN" "JST Commercial"
 			(at 167.64 69.85 0)
 			(hide yes)
@@
 			)
 		)
-		(property "Mfr" "JST Commercial"
+		(property "PN" "PH_B2B-PH-K_1x02_P2.00mm_Vertical"
+			(at 167.64 69.85 0)
+			(hide yes)
+			(show_name no)
+			(do_not_autoplace no)
+			(effects
+				(font
+					(size 1.27 1.27)
+				)
+			)
+		)
+		(property "RoHS" "By exemption"
+			(at 167.64 69.85 0)
+			(hide yes)
+			(show_name no)
+			(do_not_autoplace no)
+			(effects
+				(font
+					(size 1.27 1.27)
+				)
+			)
+		)
+		(property "Temperature" "Top = -25 °C to 85 °C"
 			(at 167.64 69.85 0)
 			(hide yes)
@@
 			)
 		)
-		(property "Description" "Luminus Devices SST-08H-UV"
+		(property "Description" "UV LED 365nm"
 			(at 114.3 83.82 0)
 			(hide yes)
@@
 			)
 		)
-		(property "MN" "SST-08-UV-A40H-F365-00 "
+		(property "Temperature" "Top = 0 °C to 100 °C"
 			(at 114.3 83.82 90)
 			(hide yes)
@@
 			)
 		)
-		(property "Mfr" "Luminus Devices"
+		(property "RoHS" "Yes"
 			(at 114.3 83.82 90)
 			(hide yes)
@@
 			)
 		)
-		(property "Temperature" "Top = 0 °C to 125 °C"
+		(property "MFN" "Luminus Devices"
 			(at 114.3 83.82 90)
 			(hide yes)
@@
 			)
 		)
-		(property "RoHS" "Yes"
+		(property "PN" "SST-08-UV-A40H-F365-00"
 			(at 114.3 83.82 90)
 			(hide yes)
@@
 			)
 		)
-		(property "Description" "Luminus Devices SST-08H-UV"
+		(property "Description" "UV LED 365nm"
 			(at 114.3 119.38 0)
-			(hide yes)
-			(show_name no)
-			(do_not_autoplace no)
-			(effects
-				(font
-					(size 1.27 1.27)
-				)
-			)
-		)
-		(property "MN" "SST-08-UV-A40H-F365-00 "
-			(at 114.3 119.38 90)
-			(hide yes)
-			(show_name no)
-			(do_not_autoplace no)
-			(effects
-				(font
-					(size 1.27 1.27)
-				)
-			)
-		)
-		(property "Mfr" "Luminus Devices"
-			(at 114.3 119.38 90)
 			(hide yes)
 			(show_name no)
@@
 		)
 		(property "RoHS" "Yes"
+			(at 114.3 119.38 90)
+			(hide yes)
+			(show_name no)
+			(do_not_autoplace no)
+			(effects
+				(font
+					(size 1.27 1.27)
+				)
+			)
+		)
+		(property "MFN" "Luminus Devices"
+			(at 114.3 119.38 90)
+			(hide yes)
+			(show_name no)
+			(do_not_autoplace no)
+			(effects
+				(font
+					(size 1.27 1.27)
+				)
+			)
+		)
+		(property "PN" "SST-08-UV-A40H-F365-00"
 			(at 114.3 119.38 90)
 			(hide yes)
@@
 		(exclude_from_sim no)
 		(in_bom no)
-		(on_board yes)
+		(on_board no)
 		(in_pos_files yes)
 		(dnp no)
@@
 		(exclude_from_sim no)
 		(in_bom no)
-		(on_board yes)
+		(on_board no)
 		(in_pos_files yes)
 		(dnp no)
