File: kicad/uv-led.kicad_sch (KiCad schematic)
At the start: 13 parts, among them J1 JST_PH_B2B-PH-K_1x02_P2.00mm_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

Commit message: updated symbol fields and added RoHs and temperature to J1 connector
Parts:
- D1: MFN (none) -> Luminus Devices; MN SST-08-UV-A40H-F365-00 -> (none); Mfr Luminus Devices -> (none); PN (none) -> SST-08-UV-A40H-F365-00; Temperature Top = 0 °C to 125 °C -> Top = 0 °C to 100 °C
- D2, D3, D4, D5: MFN (none) -> Luminus Devices; MN SST-08-UV-A40H-F365-00 -> (none); Mfr Luminus Devices -> (none); PN (none) -> SST-08-UV-A40H-F365-00
- J1: MFN (none) -> JST Commercial; MN PH_B2B-PH-K_1x02_P2.00mm_Vertical -> (none); Mfr JST Commercial -> (none); PN (none) -> PH_B2B-PH-K_1x02_P2.00mm_Vertical; RoHS (none) -> By exemption; Temperature (none) -> Top = -25 °C to 85 °C
Changed lines of the file:
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@@
 			)
 		)
-		(property "Description" "Luminus Devices SST-08H-UV"
+		(property "Description" "UV LED 365nm"
 			(at 114.3 101.6 0)
-			(hide yes)
-			(show_name no)
-			(do_not_autoplace no)
-			(effects
-				(font
-					(size 1.27 1.27)
-				)
-			)
-		)
-		(property "MN" "SST-08-UV-A40H-F365-00 "
-			(at 114.3 101.6 90)
-			(hide yes)
-			(show_name no)
-			(do_not_autoplace no)
-			(effects
-				(font
-					(size 1.27 1.27)
-				)
-			)
-		)
-		(property "Mfr" "Luminus Devices"
-			(at 114.3 101.6 90)
 			(hide yes)
 			(show_name no)
@@
 		)
 		(property "RoHS" "Yes"
+			(at 114.3 101.6 90)
+			(hide yes)
+			(show_name no)
+			(do_not_autoplace no)
+			(effects
+				(font
+					(size 1.27 1.27)
+				)
+			)
+		)
+		(property "MFN" "Luminus Devices"
+			(at 114.3 101.6 90)
+			(hide yes)
+			(show_name no)
+			(do_not_autoplace no)
+			(effects
+				(font
+					(size 1.27 1.27)
+				)
+			)
+		)
+		(property "PN" "SST-08-UV-A40H-F365-00"
 			(at 114.3 101.6 90)
 			(hide yes)
@@
 			)
 		)
-		(property "Description" "Luminus Devices SST-08H-UV"
+		(property "Description" "UV LED 365nm"
 			(at 114.3 92.71 0)
-			(hide yes)
-			(show_name no)
-			(do_not_autoplace no)
-			(effects
-				(font
-					(size 1.27 1.27)
-				)
-			)
-		)
-		(property "MN" "SST-08-UV-A40H-F365-00 "
-			(at 114.3 92.71 90)
-			(hide yes)
-			(show_name no)
-			(do_not_autoplace no)
-			(effects
-				(font
-					(size 1.27 1.27)
-				)
-			)
-		)
-		(property "Mfr" "Luminus Devices"
-			(at 114.3 92.71 90)
 			(hide yes)
 			(show_name no)
@@
 		)
 		(property "RoHS" "Yes"
+			(at 114.3 92.71 90)
+			(hide yes)
+			(show_name no)
+			(do_not_autoplace no)
+			(effects
+				(font
+					(size 1.27 1.27)
+				)
+			)
+		)
+		(property "MFN" "Luminus Devices"
+			(at 114.3 92.71 90)
+			(hide yes)
+			(show_name no)
+			(do_not_autoplace no)
+			(effects
+				(font
+					(size 1.27 1.27)
+				)
+			)
+		)
+		(property "PN" "SST-08-UV-A40H-F365-00"
 			(at 114.3 92.71 90)
 			(hide yes)
@@
 			)
 		)
-		(property "Description" "Luminus Devices SST-08H-UV"
+		(property "Description" "UV LED 365nm"
 			(at 114.3 110.49 0)
-			(hide yes)
-			(show_name no)
-			(do_not_autoplace no)
-			(effects
-				(font
-					(size 1.27 1.27)
-				)
-			)
-		)
-		(property "MN" "SST-08-UV-A40H-F365-00 "
-			(at 114.3 110.49 90)
-			(hide yes)
-			(show_name no)
-			(do_not_autoplace no)
-			(effects
-				(font
-					(size 1.27 1.27)
-				)
-			)
-		)
-		(property "Mfr" "Luminus Devices"
-			(at 114.3 110.49 90)
 			(hide yes)
 			(show_name no)
@@
 		)
 		(property "RoHS" "Yes"
+			(at 114.3 110.49 90)
+			(hide yes)
+			(show_name no)
+			(do_not_autoplace no)
+			(effects
+				(font
+					(size 1.27 1.27)
+				)
+			)
+		)
+		(property "MFN" "Luminus Devices"
+			(at 114.3 110.49 90)
+			(hide yes)
+			(show_name no)
+			(do_not_autoplace no)
+			(effects
+				(font
+					(size 1.27 1.27)
+				)
+			)
+		)
+		(property "PN" "SST-08-UV-A40H-F365-00"
 			(at 114.3 110.49 90)
 			(hide yes)
@@
 			)
 		)
-		(property "MN" "PH_B2B-PH-K_1x02_P2.00mm_Vertical"
+		(property "MFN" "JST Commercial"
 			(at 167.64 69.85 0)
 			(hide yes)
@@
 			)
 		)
-		(property "Mfr" "JST Commercial"
+		(property "PN" "PH_B2B-PH-K_1x02_P2.00mm_Vertical"
+			(at 167.64 69.85 0)
+			(hide yes)
+			(show_name no)
+			(do_not_autoplace no)
+			(effects
+				(font
+					(size 1.27 1.27)
+				)
+			)
+		)
+		(property "RoHS" "By exemption"
+			(at 167.64 69.85 0)
+			(hide yes)
+			(show_name no)
+			(do_not_autoplace no)
+			(effects
+				(font
+					(size 1.27 1.27)
+				)
+			)
+		)
+		(property "Temperature" "Top = -25 °C to 85 °C"
 			(at 167.64 69.85 0)
 			(hide yes)
@@
 			)
 		)
-		(property "Description" "Luminus Devices SST-08H-UV"
+		(property "Description" "UV LED 365nm"
 			(at 114.3 83.82 0)
 			(hide yes)
@@
 			)
 		)
-		(property "MN" "SST-08-UV-A40H-F365-00 "
+		(property "Temperature" "Top = 0 °C to 100 °C"
 			(at 114.3 83.82 90)
 			(hide yes)
@@
 			)
 		)
-		(property "Mfr" "Luminus Devices"
+		(property "RoHS" "Yes"
 			(at 114.3 83.82 90)
 			(hide yes)
@@
 			)
 		)
-		(property "Temperature" "Top = 0 °C to 125 °C"
+		(property "MFN" "Luminus Devices"
 			(at 114.3 83.82 90)
 			(hide yes)
@@
 			)
 		)
-		(property "RoHS" "Yes"
+		(property "PN" "SST-08-UV-A40H-F365-00"
 			(at 114.3 83.82 90)
 			(hide yes)
@@
 			)
 		)
-		(property "Description" "Luminus Devices SST-08H-UV"
+		(property "Description" "UV LED 365nm"
 			(at 114.3 119.38 0)
-			(hide yes)
-			(show_name no)
-			(do_not_autoplace no)
-			(effects
-				(font
-					(size 1.27 1.27)
-				)
-			)
-		)
-		(property "MN" "SST-08-UV-A40H-F365-00 "
-			(at 114.3 119.38 90)
-			(hide yes)
-			(show_name no)
-			(do_not_autoplace no)
-			(effects
-				(font
-					(size 1.27 1.27)
-				)
-			)
-		)
-		(property "Mfr" "Luminus Devices"
-			(at 114.3 119.38 90)
 			(hide yes)
 			(show_name no)
@@
 			(at 114.3 119.38 90)
 			(hide yes)
+			(show_name no)
+			(do_not_autoplace no)
+			(effects
+				(font
+					(size 1.27 1.27)
+				)
+			)
+		)
+		(property "MFN" "Luminus Devices"
+			(at 114.3 119.38 90)
+			(hide yes)
+			(show_name no)
+			(do_not_autoplace no)
+			(effects
+				(font
+					(size 1.27 1.27)
+				)
+			)
+		)
+		(property "PN" "SST-08-UV-A40H-F365-00"
+			(at 114.3 119.38 90)
+			(hide yes)

Commit message: added libraries and linked footprints
Parts:
- LOGO3: footprint Symbol:OSHW-Logo_7.5x8mm_SilkScreen -> (none)
Changed lines of the file:
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@@
 		(exclude_from_sim no)
 		(in_bom no)
-		(on_board yes)
+		(on_board no)
 		(in_pos_files yes)
 		(dnp no)
@@
 			)
 		)
-		(property "Footprint" "Symbol:OSHW-Logo_7.5x8mm_SilkScreen"
+		(property "Footprint" ""
 			(at 278.13 173.99 0)
 			(hide yes)
@@
 		(exclude_from_sim no)
 		(in_bom no)
-		(on_board yes)
+		(on_board no)
 		(in_pos_files yes)
 		(dnp no)
@@
 		(exclude_from_sim no)
 		(in_bom no)
-		(on_board yes)
-		(in_pos_files yes)
-		(dnp no)
+		(on_board no)
+		(in_pos_files yes)
+		(dnp no)

Commit message: Fixed BOM (#18)
- Fixed JST PN
- Fixed LED temperature
- Bumped to v1.1.1
Parts:
- D1, D2, D3, D4, D5: Temperature Top = 0 °C to 100 °C -> Top = -40 °C to 95 °C
- J1: Alternative (none) -> JST B2B-PH-KL(LF)(SN); PN PH_B2B-PH-K_1x02_P2.00mm_Vertical -> B2B-PH-K(LF)(SN); RoHS By exemption -> Yes
Changed lines of the file:
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@@
 		(title "QUIPS-C UV-LED")
 		(date "2026-09-02")
-		(rev "1.1.0")
+		(rev "1.1.1")
 		(company "TU Darmstadt")
 		(comment 1 "Copyright (©) 2026, Tom Güntzel <tom.guentzel@physik.tu-darmstadt.de>")
@@
 			)
 		)
-		(property "Temperature" "Top = 0 °C to 100 °C"
+		(property "Temperature" "Top = -40 °C to 95 °C"
 			(at 114.3 101.6 90)
 			(hide yes)
@@
 			)
 		)
-		(property "Temperature" "Top = 0 °C to 100 °C"
+		(property "Temperature" "Top = -40 °C to 95 °C"
 			(at 114.3 92.71 90)
 			(hide yes)
@@
 			)
 		)
-		(property "Temperature" "Top = 0 °C to 100 °C"
+		(property "Temperature" "Top = -40 °C to 95 °C"
 			(at 114.3 110.49 90)
 			(hide yes)
@@
 			)
 		)
-		(property "PN" "PH_B2B-PH-K_1x02_P2.00mm_Vertical"
+		(property "PN" "B2B-PH-K(LF)(SN)"
 			(at 167.64 69.85 0)
 			(hide yes)
@@
 			)
 		)
-		(property "RoHS" "By exemption"
+		(property "RoHS" "Yes"
 			(at 167.64 69.85 0)
 			(hide yes)
@@
 		)
 		(property "Temperature" "Top = -25 °C to 85 °C"
+			(at 167.64 69.85 0)
+			(hide yes)
+			(show_name no)
+			(do_not_autoplace no)
+			(effects
+				(font
+					(size 1.27 1.27)
+				)
+			)
+		)
+		(property "Alternative" "JST B2B-PH-KL(LF)(SN)"
 			(at 167.64 69.85 0)
 			(hide yes)
@@
 			)
 		)
-		(property "Temperature" "Top = 0 °C to 100 °C"
+		(property "Temperature" "Top = -40 °C to 95 °C"
 			(at 114.3 83.82 90)
 			(hide yes)
@@
 			)
 		)
-		(property "Temperature" "Top = 0 °C to 100 °C"
+		(property "Temperature" "Top = -40 °C to 95 °C"
 			(at 114.3 119.38 90)
 			(hide yes)

Commit message: Feature/two layer PCB with vias (#19)
* enlarged drill holes for M6 screws for more tolerance

* updated mount revision number to 1.2.0

* updated revision number to 1.2.0

* updated PCB revision label

* screw pads changed to unconnected

* updated physical stackup to two 70um copper layers

* Added missing infos

- Missing dimension
- Moved J1 label
- Added board finish

---------

Co-authored-by: Patrick Baus <patrick.baus@physik.tu-darmstadt.de>
Connections:
- net GND: no longer H1.1, H2.1
- no-connect marks 0 -> 2
Changed lines of the file:
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@@
 	(title_block
 		(title "QUIPS-C UV-LED")
-		(date "2026-09-02")
-		(rev "1.1.1")
+		(date "2026-09-30")
+		(rev "1.2.0")
 		(company "TU Darmstadt")
 		(comment 1 "Copyright (©) 2026, Tom Güntzel <tom.guentzel@physik.tu-darmstadt.de>")
@@
 		(color 0 0 0 0)
 	)
+	(no_connect
+		(at 165.1 105.41)
+	)
+	(no_connect
+		(at 139.7 105.41)
+	)
 	(wire
 		(pts
@@
 	(wire
 		(pts
-			(xy 139.7 105.41) (xy 139.7 106.68)
-		)
-		(stroke
-			(width 0)
-			(type default)
-		)
-	)
-	(wire
-		(pts
 			(xy 114.3 77.47) (xy 114.3 80.01)
-		)
-		(stroke
-			(width 0)
-			(type default)
-		)
-	)
-	(wire
-		(pts
-			(xy 165.1 105.41) (xy 165.1 106.68)
 		)
 		(stroke
@@
 	)
 	(symbol
-		(lib_id "power:GND")
-		(at 139.7 106.68 0)
-		(unit 1)
-		(body_style 1)
-		(exclude_from_sim no)
-		(in_bom yes)
-		(on_board yes)
-		(in_pos_files yes)
-		(dnp no)
-		(fields_autoplaced yes)
-		(property "Reference" "#PWR04"
-			(at 139.7 113.03 0)
-			(hide yes)
-			(show_name no)
-			(do_not_autoplace no)
-			(effects
-				(font
-					(size 1.27 1.27)
-				)
-			)
-		)
-		(property "Value" "GND"
-			(at 139.7 111.76 0)
-			(show_name no)
-			(do_not_autoplace no)
-			(effects
-				(font
-					(size 1.27 1.27)
-				)
-			)
-		)
-		(property "Footprint" ""
-			(at 139.7 106.68 0)
-			(hide yes)
-			(show_name no)
-			(do_not_autoplace no)
-			(effects
-				(font
-					(size 1.27 1.27)
-				)
-			)
-		)
-		(property "Datasheet" ""
-			(at 139.7 106.68 0)
-			(hide yes)
-			(show_name no)
-			(do_not_autoplace no)
-			(effects
-				(font
-					(size 1.27 1.27)
-				)
-			)
-		)
-		(property "Description" "Power symbol creates a global label with name \"GND\" , ground"
-			(at 139.7 106.68 0)
-			(hide yes)
-			(show_name no)
-			(do_not_autoplace no)
-			(effects
-				(font
-					(size 1.27 1.27)
-				)
-			)
-		)
-		(pin "1"
-		)
-		(instances
-			(project "uv-led"
-				(path "/e67fac83-14c9-457c-9fba-69cbeffeeea3"
-					(reference "#PWR04")
-					(unit 1)
-				)
-			)
-		)
-	)
-	(symbol
 		(lib_id "Connector_Generic:Conn_01x02")
 		(at 167.64 69.85 0)
@@
 					(unit 1)
 				)
-			)
-		)
-	)
-	(symbol
-		(lib_id "power:GND")
-		(at 165.1 106.68 0)
-		(unit 1)
-		(body_style 1)
-		(exclude_from_sim no)
-		(in_bom yes)
-		(on_board yes)
-		(in_pos_files yes)
-		(dnp no)
-		(fields_autoplaced yes)
-		(property "Reference" "#PWR03"
-			(at 165.1 113.03 0)
-			(hide yes)
-			(show_name no)
-			(do_not_autoplace no)
-			(effects
-				(font
-					(size 1.27 1.27)
-				)
-			)
-		)
-		(property "Value" "GND"
-			(at 165.1 111.76 0)
-			(show_name no)
-			(do_not_autoplace no)
-			(effects
-				(font
-					(size 1.27 1.27)
-				)
-			)
-		)
-		(property "Footprint" ""
-			(at 165.1 106.68 0)
-			(hide yes)
-			(show_name no)
-			(do_not_autoplace no)
-			(effects
-				(font
-					(size 1.27 1.27)
-				)
-			)
-		)
-		(property "Datasheet" ""
-			(at 165.1 106.68 0)
-			(hide yes)
-			(show_name no)
-			(do_not_autoplace no)
-			(effects
-				(font
-					(size 1.27 1.27)
-				)
-			)
-		)
-		(property "Description" "Power symbol creates a global label with name \"GND\" , ground"
-			(at 165.1 106.68 0)
-			(hide yes)
-			(show_name no)
-			(do_not_autoplace no)
-			(effects
-				(font
-					(size 1.27 1.27)
-				)
-			)
-		)
-		(pin "1"
-		)
-		(instances
-			(project "uv-led"
-				(path "/e67fac83-14c9-457c-9fba-69cbeffeeea3"
-					(reference "#PWR03")
-					(unit 1)
-				)
